Commit message: Update URDF model for 2 Poppy Ergo configuration.

File: hardware/URDF/Poppy_Ergo/robots/Poppy_Ergo_Flat_Support.URDF (robot description, URDF)
Before this commit: robot Poppy_Ergo_Flat_Base, 7 links, 6 joints
Links:
- link U_shape: mass 0.00600499024509973 -> 0.00558464092794276; geometry collision mesh filename=package://flat/meshes/U_shape.STL; visual mesh filename=package://flat/meshes/U_shape.STL
- link base_link: mass 0.149645525028119 -> 0.144396264939993; geometry collision mesh filename=package://flat/meshes/base_link.STL; visual mesh filename=package://flat/meshes/base_link.STL
- link base_module_2: mass 0.0804147809717077 -> 0.0801745189910368; geometry collision mesh filename=package://flat/meshes/base_module_2.STL; visual mesh filename=package://flat/meshes/base_module_2.STL
- link module_1: mass 0.0833142368972856 -> 0.0828710129889412; geometry collision mesh filename=package://flat/meshes/module_1.STL; visual mesh filename=package://flat/meshes/module_1.STL
- link tip: mass 0.0746560951391437 -> 0.0746560951328427; geometry collision mesh filename=package://flat/meshes/tip.STL; visual mesh filename=package://flat/meshes/tip.STL
- link tip_middle: mass 0.0833142368971469 -> 0.0828710129932394; geometry collision mesh filename=package://flat/meshes/tip_middle.STL; visual mesh filename=package://flat/meshes/tip_middle.STL
- link tip_module_1: mass 0.0802833119039321 -> 0.0798894067305018; geometry collision mesh filename=package://flat/meshes/tip_module_1.STL; visual mesh filename=package://flat/meshes/tip_module_1.STL
Joints:
- joint m1: origin xyz=0 0 0.0205 rpy=-6.12303176911189E-17 0 0 -> xyz=-0.000819116943949499 0 0.0395000000000191 rpy=0 0 1.5707963267949
- joint m4: origin xyz=0 0.063 0 rpy=0 0 0 -> xyz=0 0.03715 0 rpy=0 0 0
- joint m5: origin xyz=0 0 0.0702000000000001 rpy=1.5707963267949 0 0 -> xyz=0 0.0258500000000001 0.0702000000000001 rpy=1.5707963267949 0 0
- joint m6: axis 0 0 -1 -> -1 0 0; origin xyz=0 0.0699999999999999 0 rpy=0 -1.5707963267949 0 -> xyz=0 0.07 0 rpy=0 0 -9.36192041654558E-16

Commit message: fix meshes links

File: hardware/URDF/Poppy_Ergo/robots/Poppy_Ergo_Flat_Support.URDF (robot description, URDF)
Before this commit: robot flat, 7 links, 6 joints
Links:
- link U_shape: geometry collision mesh filename=package://Poppy_Ergo/meshes/U_shape.STL; visual mesh filename=package://Poppy_Ergo/meshes/U_shape.STL
- link base_link: geometry collision mesh filename=package://Poppy_Ergo/meshes/flat_base.STL; visual mesh filename=package://Poppy_Ergo/meshes/flat_base.STL
- link base_module_2: geometry collision mesh filename=package://Poppy_Ergo/meshes/base_module_2.STL; visual mesh filename=package://Poppy_Ergo/meshes/base_module_2.STL
- link module_1: geometry collision mesh filename=package://Poppy_Ergo/meshes/module_1.STL; visual mesh filename=package://Poppy_Ergo/meshes/module_1.STL
- link tip: geometry collision mesh filename=package://Poppy_Ergo/meshes/tip.STL; visual mesh filename=package://Poppy_Ergo/meshes/tip.STL
- link tip_middle: geometry collision mesh filename=package://Poppy_Ergo/meshes/tip_middle.STL; visual mesh filename=package://Poppy_Ergo/meshes/tip_middle.STL
- link tip_module_1: geometry collision mesh filename=package://Poppy_Ergo/meshes/tip_module_1.STL; visual mesh filename=package://Poppy_Ergo/meshes/tip_module_1.STL

File: hardware/URDF/Poppy_Ergo/robots/Poppy_Ergo_Suction_Pad.URDF (robot description, URDF)
Before this commit: robot Poppy_Ergo, 7 links, 6 joints
Links:
- link base_link: geometry collision mesh filename=package://Poppy_Ergo/meshes/support_suction_pad.STL; visual mesh filename=package://Poppy_Ergo/meshes/support_suction_pad.STL
